File: schematic/IH53EV.kicad_sch (KiCad schematic)
At the start: 28 parts, among them K2 T9AP1D52-12, SW1 Kill Switch HVBD6AXR, SW3 Ignition Switch, SW4 Inertia Switch, X1 GV200QA-1

Commit message: working on schematic
Parts:
- removed 2Pole_1000V_DC_10Amp, 2Pole_1000V_DC_32Amp, Circuit_Breaker, Circuit_Breaker1: (no value), symbol Switch:SW_SPST
- removed AC/DC: RAC02-12SE_277, RAC02-12SE_277:CONV_RAC02-12SE_277, symbol RAC02-12SE_277:RAC02-12SE_277
- removed DCIS_DC/DC_Convertor: (no value), symbol DCIS DC-DC Convertor:Convertor
- removed F1, F2: 5A, symbol Device:Fuse
- removed F3: F5x20 (1A max), symbol Device:Fuse
- removed J1772: (no value), symbol Thunderstuck TSM2500:J1772
- removed OrionBMS2_IO: (no value), symbol Orion_BMS:IO_Connector
- removed Power_Relay: T92P11D22-12, symbol Relay:Relay_DPST-NO
- removed R1: 120, symbol Device:R_Small_US
- removed Thunderstruck_TSM2500_Charger: (no value), symbol Thunderstuck TSM2500:Charger
- removed X1: GV200QA-1, symbol Relay:Relay_SPST-NO
- added 2Pole_1000V_DC_10Amp1, 2Pole_1000V_DC_32Amp1, Circuit_Breaker3, Circuit_Breaker4: (no value), symbol Switch:SW_SPST
- added AC/DC1: RAC02-12SE_277, RAC02-12SE_277:CONV_RAC02-12SE_277, symbol RAC02-12SE_277:RAC02-12SE_277
- added Anderson350A600V1: (no value), symbol Disconnects:Anderson_350A_600V
- added AndersonSB1: (no value), symbol Disconnects:Anderson_SB50
- added BBCANOPCanbusIsolator1: (no value), symbol Disconnects:BB_CANOP_Canbus_Isolator
- added Blue_Sea_5032: (no value), symbol blue_sea_5032:BlueSea5032
- added CANdapter1: (no value), symbol CANdapter:CANdapter
- added DCIS_DC/DC_Convertor1: (no value), symbol DCIS DC-DC Convertor:Convertor
- added DelphiWeather4Pack1: (no value), symbol Disconnects:Delphi_Weather_4_pack
- added DeutschDTM3-pin1: (no value), symbol Disconnects:Deutsch_DTM_3-pin
- added F5: MAXI 5006 80A, symbol Device:Fuse
- added F6: MAXI 5006 50A, symbol Device:Fuse
- added F7: F5x20 (1A max), symbol Device:Fuse
- added G1: GV200QA-1, symbol Relay:Relay_SPST-NO
- added J1773: (no value), symbol Thunderstuck TSM2500:J1772
- added K3: Cole Hersee 24213, symbol Relay:Relay_SPST-NO
- added K4: fix me, symbol Relay:Relay_SPST-NO
- added OrionBMS2_IO1: (no value), symbol Orion_BMS:IO_Connector
- added Power_Relay1: T92P11D22-12, symbol Relay:Relay_DPST-NO
- added TerminalBlock1: (no value), symbol TerminalBlock:Terminal_Block
- added TerminalBlock2: (no value), symbol TerminalBlock:Terminal_Block-
- added TerminalBlock3: (no value), symbol TerminalBlock:Terminal_Block+
- added Thunderstruck_TSM2500_Charger1: (no value), symbol Thunderstuck TSM2500:Charger
- added USBConnector1: (no value), symbol Disconnects:USB
- F4: value fix me -> A25X500-4
Connections:
- net GND: now also AC/DC1.3 (-VOUT), AndersonSB1., Blue_Sea_5032. (GND), J1773., K3.1, K4.1, Thunderstruck_TSM2500_Charger1.3 (AC_Input_Earth_Ground)
- net at K2.1: now also Blue_Sea_5032.6 (Ready/Precharge), DelphiWeather4Pack1.; no longer SW3.2 (B)
- net at K2.2: now also DelphiWeather4Pack1.
- net at K2.3: now also NON_ISOLATED_LOGIC_X1_CONTROLLER.K1-24 (Precharge/Key_Switch_In); no longer Circuit_Breaker2.1 (A)
- net at K2.4: now also Circuit_Breaker2.1 (A); no longer NON_ISOLATED_LOGIC_X1_CONTROLLER.K1-24 (Precharge/Key_Switch_In)
- net at SW1.1 (A): now also TerminalBlock1.; no longer Circuit_Breaker2.2 (B)
- net at NON_ISOLATED_LOGIC_X1_CONTROLLER. (B+): now also G1.A2-
- net at NON_ISOLATED_LOGIC_X1_CONTROLLER.K1-25 (COIL_RETURN_+): now also G1.X1
- net at NON_ISOLATED_LOGIC_X1_CONTROLLER.K1-26 (DRIVER_OUT_1_-): now also G1.X2
- net at NON_ISOLATED_LOGIC_X1_CONTROLLER.K1-13 (CAN_H): now also DeutschDTM3-pin1.
- net at NON_ISOLATED_LOGIC_X1_CONTROLLER.K1-2 (CAN_L): now also DeutschDTM3-pin1.
- net at SW4.1 (A): now also SW3.2 (B)
- net at SW3.1 (A): now also K3.2; no longer SW4.2 (B)
- net at BT4.: now also BT3.
- net at BT5.: now also BT6.; no longer BT4.
- net at BT3.: no longer BT4.
- net at BT2.: now also TerminalBlock2.; no longer NON_ISOLATED_LOGIC_X1_CONTROLLER. (B-)
- net at BT6.: no longer BT5.
- net at BT1.1 (+): now also F5.2, F6.1
- new net: BBCANOPCanbusIsolator1., DelphiWeather4Pack1., K4.2, OrionBMS2_IO1.2 (READY_Power)
- new net: BBCANOPCanbusIsolator1., DelphiWeather4Pack1., OrionBMS2_IO1.12 (Ground)
- new net: BBCANOPCanbusIsolator1., OrionBMS2_IO1.17 (CAN1_Sheild)
- new net: BBCANOPCanbusIsolator1., CANdapter1. (CAN_L), OrionBMS2_IO1.18 (CAN1_H), Thunderstruck_TSM2500_Charger1.6 (CAN_H)
- new net: BBCANOPCanbusIsolator1., CANdapter1. (CAN_L), OrionBMS2_IO1.19 (CAN1_L), Thunderstruck_TSM2500_Charger1.8 (CAN_L)
- new net: BBCANOPCanbusIsolator1., DeutschDTM3-pin1. (x3)
- new net: Blue_Sea_5032. (GND), DelphiWeather4Pack1.
- new net: Blue_Sea_5032.2, DelphiWeather4Pack1.
- new net: DelphiWeather4Pack1., OrionBMS2_IO1.1 (Always_On_Power)
- new net: DelphiWeather4Pack1., OrionBMS2_IO1.7 (DISCHARGE_enable)
- new net: Blue_Sea_5032. (GND), K3.3
- new net: Blue_Sea_5032. (GND), F5.1, K3.4
- new net: Blue_Sea_5032.5, SW4.2 (B)
- new net: BT4., BT5.
- new net: Anderson350A600V1., NON_ISOLATED_LOGIC_X1_CONTROLLER. (B+)
- new net: NON_ISOLATED_LOGIC_X1_CONTROLLER.K1-14 (CAN_H_RES), NON_ISOLATED_LOGIC_X1_CONTROLLER.K1-3 (CAN_L_RES)
- new net: 2Pole_1000V_DC_10Amp1.1 (A), DCIS_DC/DC_Convertor1. (Key_Switch_Control), K4.3
- new net: DCIS_DC/DC_Convertor1. (Key_Switch_Control), K4.4
- new net: Power_Relay1.13, Thunderstruck_TSM2500_Charger1.2 (AC_Input_Neutral)
- new net: AC/DC1.1 (VAC_IN(N)), J1773., Power_Relay1.14
- new net: Power_Relay1.23, Thunderstruck_TSM2500_Charger1.1 (AC_Input_Line)
- new net: F7.2, J1773., Power_Relay1.24
- new net: AC/DC1.4 (+VOUT), OrionBMS2_IO1.3 (CHARGE_Power), Power_Relay1.A1
- new net: OrionBMS2_IO1.6 (Charger_Safety_(on/off)), Power_Relay1.A2
- new net: Circuit_Breaker3.1 (A), Thunderstruck_TSM2500_Charger1.4 (DC_Output_+)
- new net: Circuit_Breaker3.2 (B), TerminalBlock1.
- new net: BT2., BT3.
- new net: AndersonSB1., F6.2
- new net: Anderson350A600V1., TerminalBlock3.
- new net: Anderson350A600V1., TerminalBlock2.
- new net: Anderson350A600V1., TerminalBlock1.
- new net: 2Pole_1000V_DC_32Amp1.1 (A), Thunderstruck_TSM2500_Charger1.5 (DC_Ouput_-)
- new net: 2Pole_1000V_DC_32Amp1.2 (B), TerminalBlock2.
- new net: G1.A1+, TerminalBlock3.
- new net: AndersonSB1., DCIS_DC/DC_Convertor1. (Key_Switch_Control) (x2)
- new net: Circuit_Breaker4.1 (A), DCIS_DC/DC_Convertor1. (Key_Switch_Control)
- new net: J1773., OrionBMS2_IO1.13 (J1772_Control_Pilot)
- new net: J1773., OrionBMS2_IO1.14 (J1772_Proximity_Detect)
- new net: CANdapter1. (CAN_L), USBConnector1.
- new net: Circuit_Breaker2.2 (B), TerminalBlock3.
- new net: AC/DC1.2 (VAC_IN(L)), F7.1
- new net: 2Pole_1000V_DC_10Amp1.2 (B), TerminalBlock2.
- new net: Circuit_Breaker4.2 (B), TerminalBlock1.
- now unconnected: BT3.
- no-connect marks 0 -> 3
Other:
- note added: "+"
- note added: "-"
- note added: "10AWG TXL"
- note added: "14AWG AC"
- note added: "18AWG 300VAC"
- note added: "18AWG TXL"
- note added: "2/0 DLO"
- note added: "22AWG TXL"
- note added: "48V"
- note added: "4AWG SGX"
- note added: "CAN Sheilding not terminated"
- note added: "CAN1 baud rate: 250Kbps"
- note added: "Vehicle Front"
- note added: "Vehicle Rear"
- note added: "WIRE KEY (AWG = size) TXL = 12V/48V primary (GXL OK, same AWG) SGX = 12V battery cable (4 AWG) HV = 600-1000V DC pack (silicone/EV) AC = J1772 / T92 mains (600V) 300VAC = RAC02 tap only DLO = traction / pack 2/0"
- note added: "internal termination"
- note added: "internally termination"
- note removed: "48v"
- moved on the sheet: BT2, BT3, BT4, BT5, BT6

Commit message: add wires.md
Connections:
- net at DeutschDTM3-pin1.: no longer BBCANOPCanbusIsolator1.
- net at DelphiWeather4Pack1.: now also OrionBMS2_IO1.7 (DISCHARGE_enable); no longer Blue_Sea_5032. (GND)
- net at Blue_Sea_5032.2: no longer DelphiWeather4Pack1.
- net at Blue_Sea_5032.5: now also SW4.2 (B)
- net at BT4.: now also BT3.
- net at BT5.: now also BT6.; no longer BT4.
- net at BT3.: no longer BT4.
- net at NON_ISOLATED_LOGIC_X1_CONTROLLER. (B+): now also G1.A2-; no longer Anderson350A600V1.
- net at 2Pole_1000V_DC_10Amp1.1 (A), DCIS_DC/DC_Convertor1. (Key_Switch_Control): no longer K4.3
- net at BT2.: now also TerminalBlock2.
- net at TerminalBlock2.: now also 2Pole_1000V_DC_10Amp1.2 (B); no longer BT2.
- net at BT6.: no longer BT5.
- net at Anderson350A600V1.: now also TerminalBlock1.; no longer TerminalBlock3.
- net at TerminalBlock1.: now also Circuit_Breaker4.2 (B); no longer Anderson350A600V1.
- net at Circuit_Breaker4.1 (A), DCIS_DC/DC_Convertor1. (Key_Switch_Control): now also K4.3
- net at TerminalBlock3.: now also Circuit_Breaker2.2 (B)
- new net: BBCANOPCanbusIsolator1., DelphiWeather4Pack1., OrionBMS2_IO1.12 (Ground)
- new net: BBCANOPCanbusIsolator1., DeutschDTM3-pin1. (x2)
- new net: Blue_Sea_5032. (GND), DelphiWeather4Pack1.
- new net: Blue_Sea_5032.2, DelphiWeather4Pack1.
- new net: Blue_Sea_5032.6 (Ready/Precharge), DelphiWeather4Pack1., K2.1
- new net: BT4., BT5.
- new net: Anderson350A600V1., NON_ISOLATED_LOGIC_X1_CONTROLLER. (B+)
- new net: BT2., BT3.
- new net: Anderson350A600V1., TerminalBlock3.
- new net: Anderson350A600V1., TerminalBlock2.
- new net: AndersonSB1., DCIS_DC/DC_Convertor1. (Key_Switch_Control) (x2)
- now unconnected: BT3., Blue_Sea_5032.6 (Ready/Precharge), DeutschDTM3-pin1.
Other:
- moved on the sheet: 2Pole_1000V_DC_32Amp1, Circuit_Breaker2, Circuit_Breaker3, G1, K2, NON_ISOLATED_LOGIC_X1_CONTROLLER, TerminalBlock3

Commit message: checkpint
Parts:
- removed AndersonSB1: (no value), symbol Disconnects:Anderson_SB50
- added AndersonSB50: (no value), symbol Disconnects:Anderson_SB50
- added DJ7021-8-1: (no value), symbol Disconnects:DJ7021-8-21
- added DJ7031-4.8: (no value), symbol Disconnects:DJ7031-4.8
- added dj70310-6.3-1: (no value), symbol Disconnects:dj70310-6.3-11
- F5: value MAXI 5006 80A -> MAXI 5006 50A
- K4: value fix me -> G9EJ-1-E-UVD DC12
Connections:
- net GND: now also DJ7021-8-1., DJ7031-4.8.; no longer Thunderstruck_TSM2500_Charger1.3 (AC_Input_Earth_Ground)
- net at DeutschDTM3-pin1.: no longer BBCANOPCanbusIsolator1.
- net at DelphiWeather4Pack1.: now also OrionBMS2_IO1.7 (DISCHARGE_enable); no longer Blue_Sea_5032. (GND)
- net at Blue_Sea_5032.2: no longer DelphiWeather4Pack1.
- net at Blue_Sea_5032.5: now also SW4.2 (B)
- net at BT4.: now also BT3.
- net at BT5.: now also BT6.; no longer BT4.
- net at BT3.: no longer BT4.
- net at NON_ISOLATED_LOGIC_X1_CONTROLLER. (B+): now also G1.A2-; no longer Anderson350A600V1.
- net at Circuit_Breaker4.1 (A), K4.3: now also dj70310-6.3-1.; no longer DCIS_DC/DC_Convertor1. (Key_Switch_Control)
- net at K4.4: now also dj70310-6.3-1.; no longer DCIS_DC/DC_Convertor1. (Key_Switch_Control)
- net at Power_Relay1.13: now also DJ7031-4.8.; no longer Thunderstruck_TSM2500_Charger1.2 (AC_Input_Neutral)
- net at Power_Relay1.23: now also DJ7031-4.8.; no longer Thunderstruck_TSM2500_Charger1.1 (AC_Input_Line)
- net at Circuit_Breaker3.1 (A): now also TerminalBlock2.; no longer Thunderstruck_TSM2500_Charger1.4 (DC_Output_+)
- net at Circuit_Breaker3.2 (B): now also AndersonSB50.; no longer TerminalBlock1.
- net at BT2.: now also TerminalBlock2.
- net at TerminalBlock2.: now also 2Pole_1000V_DC_10Amp1.2 (B); no longer BT2.
- net at F6.2: now also DJ7021-8-1.
- net at BT6.: no longer BT5.
- net at Anderson350A600V1.: now also TerminalBlock1.; no longer TerminalBlock3.
- net at TerminalBlock1.: now also Circuit_Breaker4.2 (B); no longer Anderson350A600V1.
- net at Thunderstruck_TSM2500_Charger1.5 (DC_Ouput_-): now also AndersonSB50.; no longer 2Pole_1000V_DC_32Amp1.1 (A)
- net at 2Pole_1000V_DC_32Amp1.2 (B): now also AndersonSB50.; no longer TerminalBlock2.
- net at DCIS_DC/DC_Convertor1. (Key_Switch_Control): now also DJ7021-8-1.
- net at 2Pole_1000V_DC_10Amp1.1 (A): now also dj70310-6.3-1.; no longer DCIS_DC/DC_Convertor1. (Key_Switch_Control)
- net at TerminalBlock3.: now also Circuit_Breaker2.2 (B)
- new net: BBCANOPCanbusIsolator1., DelphiWeather4Pack1., OrionBMS2_IO1.12 (Ground)
- new net: BBCANOPCanbusIsolator1., DeutschDTM3-pin1. (x2)
- new net: Blue_Sea_5032. (GND), DelphiWeather4Pack1.
- new net: Blue_Sea_5032.2, DelphiWeather4Pack1.
- new net: Blue_Sea_5032.6 (Ready/Precharge), DelphiWeather4Pack1., K2.1
- new net: BT4., BT5.
- new net: Anderson350A600V1., NON_ISOLATED_LOGIC_X1_CONTROLLER. (B+)
- new net: BT2., BT3.
- new net: Anderson350A600V1., TerminalBlock3.
- new net: Anderson350A600V1., TerminalBlock2.
- new net: AndersonSB50., Thunderstruck_TSM2500_Charger1.4 (DC_Output_+)
- new net: 2Pole_1000V_DC_32Amp1.1 (A), TerminalBlock1.
- new net: DCIS_DC/DC_Convertor1. (Key_Switch_Control), dj70310-6.3-1. (x3)
- new net: DCIS_DC/DC_Convertor1. (Key_Switch_Control), DJ7021-8-1.
- new net: DJ7031-4.8., Thunderstruck_TSM2500_Charger1.1 (AC_Input_Line)
- new net: DJ7031-4.8., Thunderstruck_TSM2500_Charger1.2 (AC_Input_Neutral)
- new net: DJ7031-4.8., Thunderstruck_TSM2500_Charger1.3 (AC_Input_Earth_Ground)
- now unconnected: BT3., Blue_Sea_5032.6 (Ready/Precharge), DeutschDTM3-pin1.
Other:
- note added: "10 AWG HV"
- note added: "10AWG GLX"
- note added: "10AWG HV"
- note added: "18AWG AC"
- note added: "18AWG HV"
- note added: "WIRE KEY (AWG = size) TXL = 12V/48V primary (GXL OK, same AWG) SGX = 12V battery cable (10 AWG) HV = 600-1000V DC pack (silicone/EV) AC = J1772 / T92 mains (600V) 300VAC = RAC02 tap only DLO = traction / pack 2/0"
- note removed: "10AWG TXL"
- note removed: "22AWG TXL"
- note removed: "4AWG SGX"
- note removed: "WIRE KEY (AWG = size) TXL = 12V/48V primary (GXL OK, same AWG) SGX = 12V battery cable (4 AWG) HV = 600-1000V DC pack (silicone/EV) AC = J1772 / T92 mains (600V) 300VAC = RAC02 tap only DLO = traction / pack 2/0"
- note removed: "internally termination"
- moved on the sheet: 2Pole_1000V_DC_10Amp1, 2Pole_1000V_DC_32Amp1, AC/DC1, BT1, BT2, BT3, BT4, BT5, BT6, Circuit_Breaker3, Circuit_Breaker4, DCIS_DC/DC_Convertor1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

Commit message: 3d printing to get it right
Connections:
- net at DeutschDTM3-pin1.: no longer BBCANOPCanbusIsolator1.
- net at DelphiWeather4Pack1.: now also OrionBMS2_IO1.7 (DISCHARGE_enable); no longer Blue_Sea_5032. (GND)
- net at Blue_Sea_5032.2: no longer DelphiWeather4Pack1.
- net at Blue_Sea_5032.5: now also SW4.2 (B)
- net at BT4.: now also BT3.
- net at BT5.: now also BT6.; no longer BT4.
- net at BT3.: no longer BT4.
- net at NON_ISOLATED_LOGIC_X1_CONTROLLER. (B+): now also G1.A2-; no longer Anderson350A600V1.
- net at BT2.: now also TerminalBlock2.
- net at TerminalBlock2.: now also 2Pole_1000V_DC_10Amp1.2 (B); no longer BT2.
- net at BT6.: no longer BT5.
- net at Anderson350A600V1.: now also TerminalBlock1.; no longer TerminalBlock3.
- net at TerminalBlock1.: now also Circuit_Breaker4.2 (B); no longer Anderson350A600V1.
- net at DCIS_DC/DC_Convertor1. (Key_Switch_Control): now also DJ7021-8-1.; no longer dj70310-6.3-1.
- net at dj70310-6.3-1.: now also 2Pole_1000V_DC_10Amp1.1 (A); no longer DCIS_DC/DC_Convertor1. (Key_Switch_Control)
- net at TerminalBlock3.: now also Circuit_Breaker2.2 (B)
- new net: BBCANOPCanbusIsolator1., DelphiWeather4Pack1., OrionBMS2_IO1.12 (Ground)
- new net: BBCANOPCanbusIsolator1., DeutschDTM3-pin1. (x2)
- new net: Blue_Sea_5032. (GND), DelphiWeather4Pack1.
- new net: Blue_Sea_5032.2, DelphiWeather4Pack1.
- new net: Blue_Sea_5032.6 (Ready/Precharge), DelphiWeather4Pack1., K2.1
- new net: BT4., BT5.
- new net: Anderson350A600V1., NON_ISOLATED_LOGIC_X1_CONTROLLER. (B+)
- new net: BT2., BT3.
- new net: Anderson350A600V1., TerminalBlock3.
- new net: Anderson350A600V1., TerminalBlock2.
- new net: DCIS_DC/DC_Convertor1. (Key_Switch_Control), dj70310-6.3-1. (x3)
- new net: DCIS_DC/DC_Convertor1. (Key_Switch_Control), DJ7021-8-1.
- now unconnected: BT3., Blue_Sea_5032.6 (Ready/Precharge), DeutschDTM3-pin1.
Changed lines of the file:
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@@
 	(title_block
 		(title "1953 International EV Conversion")
+		(date "2026-08-24")
 	)
 	(text "18AWG TXL"

Commit message: add AC enclosure and bus bars
Parts:
- removed TerminalBlock1: (no value), symbol TerminalBlock:Terminal_Block
- added TerminalBlock1: (no value), symbol TerminalBlock:Terminal_Block+
Connections:
- net at DeutschDTM3-pin1.: no longer BBCANOPCanbusIsolator1.
- net at DelphiWeather4Pack1.: now also OrionBMS2_IO1.7 (DISCHARGE_enable); no longer Blue_Sea_5032. (GND)
- net at Blue_Sea_5032.2: no longer DelphiWeather4Pack1.
- net at Blue_Sea_5032.5: now also SW4.2 (B)
- net at BT4.: now also BT3.
- net at BT5.: now also BT6.; no longer BT4.
- net at BT3.: no longer BT4.
- net at NON_ISOLATED_LOGIC_X1_CONTROLLER. (B+): now also G1.A2-; no longer Anderson350A600V1.
- net at BT2.: now also TerminalBlock2.
- net at TerminalBlock2.: now also 2Pole_1000V_DC_10Amp1.2 (B); no longer BT2.
- net at BT6.: no longer BT5.
- net at Anderson350A600V1.: now also TerminalBlock2.; no longer TerminalBlock3.
- net at SW1.1 (A): now also TerminalBlock1.
- net at 2Pole_1000V_DC_32Amp1.1 (A): now also TerminalBlock1.
- net at DCIS_DC/DC_Convertor1. (Key_Switch_Control): now also DJ7021-8-1.; no longer dj70310-6.3-1.
- net at dj70310-6.3-1.: now also 2Pole_1000V_DC_10Amp1.1 (A); no longer DCIS_DC/DC_Convertor1. (Key_Switch_Control)
- net at TerminalBlock3.: now also Circuit_Breaker2.2 (B)
- net at Circuit_Breaker4.2 (B): now also TerminalBlock1.
- new net: BBCANOPCanbusIsolator1., DelphiWeather4Pack1., OrionBMS2_IO1.12 (Ground)
- new net: BBCANOPCanbusIsolator1., DeutschDTM3-pin1. (x2)
- new net: Blue_Sea_5032. (GND), DelphiWeather4Pack1.
- new net: Blue_Sea_5032.2, DelphiWeather4Pack1.
- new net: Blue_Sea_5032.6 (Ready/Precharge), DelphiWeather4Pack1., K2.1
- new net: BT4., BT5.
- new net: Anderson350A600V1., NON_ISOLATED_LOGIC_X1_CONTROLLER. (B+)
- new net: BT2., BT3.
- new net: Anderson350A600V1., TerminalBlock3.
- new net: Anderson350A600V1., TerminalBlock1.
- new net: DCIS_DC/DC_Convertor1. (Key_Switch_Control), dj70310-6.3-1. (x3)
- new net: DCIS_DC/DC_Convertor1. (Key_Switch_Control), DJ7021-8-1.
- now unconnected: BT3., Blue_Sea_5032.6 (Ready/Precharge), DeutschDTM3-pin1.
Changed lines of the file:
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@@
+	)
+	(symbol
+		(lib_name "Terminal_Block+_1")
+		(lib_id "TerminalBlock:Terminal_Block+")
+		(at 469.9 243.84 0)
+		(unit 1)
+		(body_style 1)
+		(exclude_from_sim no)
+		(in_bom yes)
+		(on_board yes)
+		(in_pos_files yes)
+		(dnp no)
+		(fields_autoplaced yes)
+		(property "Reference" "TerminalBlock1"
+			(at 469.9 266.7 0)
+			(show_name no)
+			(do_not_autoplace no)
+			(effects
+				(font
+					(size 1.27 1.27)
+				)
+			)
+		)
+		(property "Value" ""
+			(at 469.9 243.84 0)
+			(show_name no)
+			(do_not_autoplace no)
+			(effects
+				(font
+					(size 1.27 1.27)
+				)
+			)
+		)
+		(property "Footprint" ""
+			(at 469.9 243.84 0)
+			(hide yes)
+			(show_name no)
+			(do_not_autoplace no)
+			(effects
+				(font
+					(size 1.27 1.27)
+				)
+			)
+		)
+		(property "Datasheet" ""
+			(at 469.9 243.84 0)
+			(hide yes)
+			(show_name no)
+			(do_not_autoplace no)
+			(effects
+				(font
+					(size 1.27 1.27)
+				)
+			)
+		)
+		(property "Description" ""
+			(at 469.9 243.84 0)
+			(hide yes)
+			(show_name no)
+			(do_not_autoplace no)
+			(effects
+				(font
+					(size 1.27 1.27)
+				)
+			)
+		)
+		(pin ""
+		)
+		(pin ""
+		)
+		(pin ""
+		)
+		(pin ""
+		)
+		(instances
+			(project "IH53EV"
+				(path "/20bcdb30-6107-4dbd-a268-7abc52ed82ed"
+					(reference "TerminalBlock1")
+					(unit 1)
+				)
+			)
+		)
 	)
 	(symbol
@@
 					(unit 1)
 				)
-			)
-		)
-	)
-	(symbol
-		(lib_id "TerminalBlock:Terminal_Block")
-		(at 469.9 243.84 0)
-		(unit 1)
-		(body_style 1)
-		(exclude_from_sim no)
-		(in_bom yes)
-		(on_board yes)
-		(in_pos_files yes)
-		(dnp no)
-		(fields_autoplaced yes)
-		(property "Reference" "TerminalBlock1"
-			(at 469.9 266.7 0)
-			(show_name no)
-			(do_not_autoplace no)
-			(effects
-				(font
-					(size 1.27 1.27)
-				)
-			)
-		)
-		(property "Value" ""
-			(at 469.9 243.84 0)
-			(show_name no)
-			(do_not_autoplace no)
-			(effects
-				(font
-					(size 1.27 1.27)
-				)
-			)
-		)
-		(property "Footprint" ""
-			(at 469.9 243.84 0)
-			(hide yes)
-			(show_name no)
-			(do_not_autoplace no)
-			(effects
-				(font
-					(size 1.27 1.27)
-				)
-			)
-		)
-		(property "Datasheet" ""
-			(at 469.9 243.84 0)
-			(hide yes)
-			(show_name no)
-			(do_not_autoplace no)
-			(effects
-				(font
-					(size 1.27 1.27)
-				)
-			)
-		)
-		(property "Description" ""
-			(at 469.9 243.84 0)
-			(hide yes)
-			(show_name no)
-			(do_not_autoplace no)
-			(effects
-				(font
-					(size 1.27 1.27)
-				)
-			)
-		)
-		(pin ""
-		)
-		(pin ""
-		)
-		(pin ""
-		)
-		(pin ""
-		)
-		(instances
-			(project "IH53EV"
-				(path "/20bcdb30-6107-4dbd-a268-7abc52ed82ed"
-					(reference "TerminalBlock1")
-					(unit 1)
-				)
