File: schematic/IH53EV.kicad_sch (KiCad schematic)
At the start: 46 parts, among them K2 T9AP1D52-12, K3 Cole Hersee 24213, K4 G9EJ-1-E-UVD DC12, SW1 Kill Switch HVBD6AXR, SW3 Ignition Switch, SW4 Inertia Switch, SW5 Instruments

Commit message: futzing with bus bar
Connections:
- net at DeutschDTM3-pin1.: no longer BBCANOPCanbusIsolator1.
- net at DelphiWeather4Pack1.: now also OrionBMS2_IO1.7 (DISCHARGE_enable); no longer Blue_Sea_5032. (GND)
- net at Blue_Sea_5032.2: no longer DelphiWeather4Pack1.
- net at Blue_Sea_5032.4: now also SW5.1 (A)
- net at Blue_Sea_5032.5: now also SW4.2 (B)
- net at BT4.: now also BT3.
- net at BT5.: now also BT6.; no longer BT4.
- net at BT3.: no longer BT4.
- net at NON_ISOLATED_LOGIC_X1_CONTROLLER. (B+): now also G1.A2-; no longer Anderson350A600V1.
- net at BT2.: now also TerminalBlock2.
- net at TerminalBlock2.: now also 2Pole_1000V_DC_10Amp1.2 (B); no longer BT2.
- net at BT6.: no longer BT5.
- net at Anderson350A600V1.: now also TerminalBlock2.; no longer TerminalBlock3.
- net at TerminalBlock1.: now also Circuit_Breaker4.2 (B); no longer Anderson350A600V1.
- net at DCIS_DC/DC_Convertor1. (Key_Switch_Control): now also DJ7021-8-1.; no longer dj70310-6.3-1.
- net at dj70310-6.3-1.: now also 2Pole_1000V_DC_10Amp1.1 (A); no longer DCIS_DC/DC_Convertor1. (Key_Switch_Control)
- net at TerminalBlock3.: now also Circuit_Breaker2.2 (B)
- new net: BBCANOPCanbusIsolator1., DelphiWeather4Pack1., OrionBMS2_IO1.12 (Ground)
- new net: BBCANOPCanbusIsolator1., DeutschDTM3-pin1. (x2)
- new net: OrionBMSCurrentSensor. (High_Channel), OrionCurrentSensor1. (High_Channel) (x3)
- new net: Blue_Sea_5032. (GND), DelphiWeather4Pack1.
- new net: Blue_Sea_5032.2, DelphiWeather4Pack1.
- new net: Blue_Sea_5032.6 (Ready/Precharge), DelphiWeather4Pack1., K2.1
- new net: BT4., BT5.
- new net: Anderson350A600V1., NON_ISOLATED_LOGIC_X1_CONTROLLER. (B+)
- new net: BT2., BT3.
- new net: Anderson350A600V1., TerminalBlock3.
- new net: Anderson350A600V1., TerminalBlock1.
- new net: DCIS_DC/DC_Convertor1. (Key_Switch_Control), dj70310-6.3-1. (x3)
- new net: DCIS_DC/DC_Convertor1. (Key_Switch_Control), DJ7021-8-1.
- now unconnected: BT3., Blue_Sea_5032.6 (Ready/Precharge), DeutschDTM3-pin1.
